File: gaia-gate.sch (KiCad schematic (older format))
At the start: 15 parts, among them J1 Conn_01x02_Male, J2 Conn_01x06_Male, J3 Conn_01x03, J4 Conn_01x06_Male, J5 Conn_01x02_Male, J6 Conn_01x01_Male, J7 Conn_01x01_Male, U1 Vcc_one_supply, U2 ATmega328P-PU, Y1 Crystal

Commit message: v2 withcontrol board circuit
Parts:
- removed J1, J5: Conn_01x02_Male, Connector_JST:JST_EH_S2B-EH_1x02_P2.50mm_Horizontal, symbol Connector:Conn_01x02_Male
- removed J2, J4: Conn_01x06_Male, Connector_JST:JST_EH_S6B-EH_1x06_P2.50mm_Horizontal, symbol Connector:Conn_01x06_Male
- removed J6, J7: Conn_01x01_Male, Connector:Banana_Jack_1Pin, symbol Connector:Conn_01x01_Male
- added D1, D2: 1N4007, Diode_THT:D_DO-41_SOD81_P10.16mm_Horizontal, symbol Diode:1N4007
- added D3, D4, D5: GREEN, LED_THT:LED_D5.0mm, symbol Device:LED
- added F1, F2: Fuse, gaia-gate:Fuse, symbol Device:Fuse
- added J1: motor, Connector_Molex:Molex_KK-396_A-41791-0003_1x03_P3.96mm_Vertical, symbol Connector:Conn_01x03_Male
- added J2: 230V_IN, Connector_Molex:Molex_KK-396_A-41791-0002_1x02_P3.96mm_Vertical, symbol Connector:Conn_01x02_Male
- added J3: Control_Signal_IN, Connector_Molex:Molex_KK-396_A-41791-0003_1x03_P3.96mm_Vertical, symbol Connector:Conn_01x03_Male
- added J5: Extras, Connector_Molex:Molex_KK-396_A-41791-0003_1x03_P3.96mm_Vertical, symbol Connector:Conn_01x03_Male
- added J6: extra_analog, Connector_Molex:Molex_KK-396_A-41791-0004_1x04_P3.96mm_Vertical, symbol Connector:Conn_01x04_Male
- added K1, K2: SANYOU_SRD_Form_C, Relay_THT:Relay_SPDT_SANYOU_SRD_Series_Form_C, symbol Relay:SANYOU_SRD_Form_C
- added Q1, Q2: BC547, Package_TO_SOT_THT:TO-92_Inline_Wide, symbol Transistor_BJT:BC547
- added R1, R2: 1K, gaia-gate:resistor, symbol Device:R
- added R3, R4, R5: 330Ω, gaia-gate:resistor, symbol Device:R
- added RV1: Varistor, Varistor:RV_Disc_D9mm_W6.1mm_P5mm, symbol Device:Varistor
- C1: renamed from C3; footprint Capacitor_THT:CP_Radial_D5.0mm_P2.50mm -> Capacitor_THT:CP_Radial_D8.0mm_P5.00mm
- C2: renamed from C1; footprint Capacitor_THT:CP_Radial_D5.0mm_P2.00mm -> Capacitor_THT:C_Disc_D3.8mm_W2.6mm_P2.50mm
- C3: renamed from C2; footprint Capacitor_THT:CP_Radial_D5.0mm_P2.00mm -> Capacitor_THT:C_Disc_D3.8mm_W2.6mm_P2.50mm
- J4: renamed from J3; footprint Connector_JST:JST_EH_S3B-EH_1x03_P2.50mm_Horizontal -> Connector_Molex:Molex_KK-396_A-41791-0003_1x03_P3.96mm_Vertical
- R6: renamed from R1; footprint Resistor_THT:R_Axial_DIN0207_L6.3mm_D2.5mm_P10.16mm_Horizontal -> gaia-gate:resistor
- R7: renamed from R2; footprint Resistor_THT:R_Axial_DIN0207_L6.3mm_D2.5mm_P10.16mm_Horizontal -> gaia-gate:resistor
- U1: footprint gaia-gate:VREG_230Vac_to_5Vdc -> gaia-gate:230_5V_supply_HiLink
- U2: footprint Package_DIP:DIP-28_W7.62mm -> Package_DIP:DIP-28_W7.62mm_Socket_LongPads
Connections:
- net labels added: AC, NEUT, Relay1_IN, Relay2_IN
- wire segments 60 -> 119
Other:
- moved on the sheet: C1, C2, C3, J4, R6, R7, U1, U2, Y1

Commit message: working PCB v2
Parts:
- removed J3: Control_Signal_IN, Connector_Molex:Molex_KK-396_A-41791-0003_1x03_P3.96mm_Vertical, symbol Connector:Conn_01x03_Male
- removed J5: Extras, Connector_Molex:Molex_KK-396_A-41791-0003_1x03_P3.96mm_Vertical, symbol Connector:Conn_01x03_Male
- added C4: 100uF, Capacitor_THT:CP_Radial_D8.0mm_P5.00mm, symbol Device:CP
- added D6: 1N4007, Diode_THT:D_DO-41_SOD81_P10.16mm_Horizontal, symbol Diode:1N4007
- added D7: GREEN, LED_THT:LED_D5.0mm, symbol Device:LED
- added J5: Extras, Connector_Molex:Molex_KK-254_AE-6410-04A_1x04_P2.54mm_Vertical, symbol Connector:Conn_01x04_Male
- added R8: 1K, gaia-gate:resistor, symbol Device:R
- added R9: 330Ω, gaia-gate:resistor, symbol Device:R
- added RV2: R_POT, Potentiometer_THT:Potentiometer_Bourns_3296W_Vertical, symbol Device:R_POT
- added U3: Current_Transformer, gaia-gate:Current_Transformer, symbol gaia_library:Current_Transformer
- added U4: LM741, Package_DIP:DIP-8_W10.16mm_LongPads, symbol Amplifier_Operational:LM741
- C1: value CP -> 10uF
- C2, C3: value C -> 0.1uf
- J3: renamed from J6; value extra_analog -> Home_Controller; footprint Connector_Molex:Molex_KK-396_A-41791-0004_1x04_P3.96mm_Vertical -> Connector_Molex:Molex_KK-254_AE-6410-04A_1x04_P2.54mm_Vertical
- J4: value Conn_01x03 -> Open_Close_Sensor; footprint Connector_Molex:Molex_KK-396_A-41791-0003_1x03_P3.96mm_Vertical -> Connector_Molex:Molex_KK-254_AE-6410-03A_1x03_P2.54mm_Vertical
- R6, R7: value 100K -> 10K
Connections:
- net +5V: now also RV2.3, U4.7 (V+); no longer J3.1 (Pin_1)
- net GND: now also J3.1 (Pin_1), C4.2, D7.1 (K), R8.2, RV2.1, U3.1 (GND), U4.4 (V-); no longer J3.4 (Pin_4)
- net NEUT: now also U3.4 (Input_Current); no longer F1.1
- net Relay1_IN: now also U2.18 (PB4); no longer U2.17 (PB3)
- net Relay2_IN: now also U2.17 (PB3)
- net Overload_Detection: now reaches U2.2 (PD0)
- net Overload_Detection: now also R9.1, U4.6
- net at U2.23 (PC0): now also J3.2 (Pin_2)
- net at U2.24 (PC1): now also J3.3 (Pin_3)
- net at U2.27 (PC4): now also J3.4 (Pin_4); no longer J3.3 (Pin_3)
- net at U2.28 (PC5): no longer J3.2 (Pin_2)
- net at U2.3 (PD1): now also J5.1 (Pin_1)
- net at U2.4 (PD2): now also J5.2 (Pin_2)
- net at U2.5 (PD3): now also J5.3 (Pin_3)
- net at U2.6 (PD4): now also J5.4 (Pin_4)
- new net: D6.2 (A), U3.2 (Signal)
- new net: C4.1, D6.1 (K), R8.1, U4.3 (+)
- new net: RV2.2, U4.2 (-)
- new net: D7.2 (A), R9.2
- new net CT_OUT: F1.1, U3.3 (Output_Current)
Other:
- moved on the sheet: C2, C3, D1, D2, D3, D4, F1, J1, J3, J4, K1, K2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

Commit message: latest pcb
Parts:
- removed C1: 10uF, Capacitor_THT:CP_Radial_D8.0mm_P5.00mm, symbol Device:CP
- removed C2, C3: 0.1uf, Capacitor_THT:C_Disc_D3.8mm_W2.6mm_P2.50mm, symbol Device:C
- removed C4: 100uF, Capacitor_THT:CP_Radial_D8.0mm_P5.00mm, symbol Device:CP
- removed D1, D2, D6: 1N4007, Diode_THT:D_DO-41_SOD81_P10.16mm_Horizontal, symbol Diode:1N4007
- removed D3, D4, D5, D7: GREEN, LED_THT:LED_D5.0mm, symbol Device:LED
- removed F1, F2: Fuse, gaia-gate:Fuse, symbol Device:Fuse
- removed J1: motor, Connector_Molex:Molex_KK-396_A-41791-0003_1x03_P3.96mm_Vertical, symbol Connector:Conn_01x03_Male
- removed J2: 230V_IN, Connector_Molex:Molex_KK-396_A-41791-0002_1x02_P3.96mm_Vertical, symbol Connector:Conn_01x02_Male
- removed J3: Home_Controller, Connector_Molex:Molex_KK-254_AE-6410-04A_1x04_P2.54mm_Vertical, symbol Connector:Conn_01x04_Male
- removed J4: Open_Close_Sensor, Connector_Molex:Molex_KK-254_AE-6410-03A_1x03_P2.54mm_Vertical, symbol Connector_Generic:Conn_01x03
- removed J5: Extras, Connector_Molex:Molex_KK-254_AE-6410-04A_1x04_P2.54mm_Vertical, symbol Connector:Conn_01x04_Male
- removed K1, K2: SANYOU_SRD_Form_C, Relay_THT:Relay_SPDT_SANYOU_SRD_Series_Form_C, symbol Relay:SANYOU_SRD_Form_C
- removed Q1, Q2: BC547, Package_TO_SOT_THT:TO-92_Inline_Wide, symbol Transistor_BJT:BC547
- removed R1, R2, R8: 1K, gaia-gate:resistor, symbol Device:R
- removed R3, R4, R5, R9: 330Ω, gaia-gate:resistor, symbol Device:R
- removed R6, R7: 10K, gaia-gate:resistor, symbol Device:R
- removed RV1: Varistor, Varistor:RV_Disc_D9mm_W6.1mm_P5mm, symbol Device:Varistor
- removed RV2: R_POT, Potentiometer_THT:Potentiometer_Bourns_3296W_Vertical, symbol Device:R_POT
- removed U1: Vcc_one_supply, gaia-gate:230_5V_supply_HiLink, symbol pcb_power_supply:Vcc_one_supply
- removed U2: ATmega328P-PU, Package_DIP:DIP-28_W7.62mm_Socket_LongPads, symbol MCU_Microchip_ATmega:ATmega328P-PU
- removed U3: Current_Transformer, gaia-gate:Current_Transformer, symbol gaia_library:Current_Transformer
- removed U4: LM741, Package_DIP:DIP-8_W10.16mm_LongPads, symbol Amplifier_Operational:LM741
- removed Y1: Crystal, Crystal:Crystal_HC18-U_Vertical, symbol Device:Crystal
